Commit message: feat: add Meca500 full stack + URDF import skills + UR5e URDF fix
Phase B4: Meca500 full stack (Demo + Sandbox + RobotControl)
- TemplateMeca500: DH 6-axis (d1=0.091, a2=0.135, a5=0.120, d6=0.070)
- MockMecademicClient, Meca500PosePresets, Meca500RobotControlTemplateDefinition
- DAE meshes 7 files from mecademic-ros2 community repo
- URDF import with URP Lit material auto-replacement
- 11 EditMode tests

UR5e URDF fix: corrected joint origins from official UR config
(roll/pitch/yaw + visual mesh offsets from visual_parameters.yaml)

URP Material pipeline: ReplaceWithUrpLitMaterials saves .mat assets
to Materials_URP/ folder, prefabs reference persisted assets

New skills: robot-urdf-import (#21), robot-control-add (#22)

Co-Authored-By: Claude Opus 4.6 (1M context) <noreply@anthropic.com>

File: Assets/Runtime/Robots/UR5e/ur5e.urdf (robot description, URDF)
Before this commit: robot ur5e, 7 links, 6 joints
Joints:
- joint shoulder_lift_joint: origin xyz=0 0 0 rpy=0 1.5707963267948966 0 -> xyz=0 0 0 rpy=1.5707963267948966 0 0
- joint wrist_1_joint: origin xyz=-0.3922 0 0.1333 rpy=0 1.5707963267948966 0 -> xyz=-0.3922 0 0.1333 rpy=0 0 0
- joint wrist_2_joint: origin xyz=0 -0.0997 0 rpy=0 -1.5707963267948966 0 -> xyz=0 -0.0997 0 rpy=1.5707963267948966 0 0
- joint wrist_3_joint: origin xyz=0 0.0996 0 rpy=0 0 0 -> xyz=0 0.0996 0 rpy=1.5707963267948966 3.141592653589793 3.141592653589793
